Commit message: 跑通rviz2

File: src/arm_moveit_config/config/ar3.ros2_control.xacro (robot description, xacro)
@@ -1,42 +1,53 @@
 <?xml version="1.0"?>
 <robot xmlns:xacro="http://www.ros.org/wiki/xacro">
-    <xacro:macro name="ar3_ros2_control" params="name">
+    <xacro:macro name="ar3_ros2_control" params="name initial_positions_file">
+        <xacro:property name="initial_positions" value="${xacro.load_yaml(initial_positions_file)['initial_positions']}"/>
         <ros2_control name="${name}" type="system">
             <hardware>
+                <!-- By default, set up controllers for simulation. This won't work on real hardware -->
+                <!--mock_components/GenericSystem 和 gazebo_ros2_control/GazeboSystem-->
                 <plugin>gazebo_ros2_control/GazeboSystem</plugin>
             </hardware>
             <joint name="joint_1">
                 <command_interface name="position"/>
-                <command_interface name="effort"/>
-                <state_interface name="position"/>
-                <state_interface name="effort"/>
+                <state_interface name="position">
+                  <param name="initial_value">${initial_positions['joint_1']}</param>
+                </state_interface>
+                <state_interface name="velocity"/>
             </joint>
             <joint name="joint_2">
                 <command_interface name="position"/>
-                <command_interface name="effort"/>
                 <state_interface name="position">
+                  <param name="initial_value">${initial_positions['joint_2']}</param>
                 </state_interface>
-                <state_interface name="effort"/>
+                <state_interface name="velocity"/>
             </joint>
             <joint name="joint_3">
                 <command_interface name="position"/>
-                <command_interface name="effort"/>
                 <state_interface name="position">
+                  <param name="initial_value">${initial_positions['joint_3']}</param>
                 </state_interface>
-                <state_interface name="effort"/>
+                <state_interface name="velocity"/>
             </joint>
             <joint name="joint_4">
                 <command_interface name="position"/>
-                <command_interface name="effort"/>
                 <state_interface name="position">
+                  <param name="initial_value">${initial_positions['joint_4']}</param>
                 </state_interface>
-                <state_interface name="effort"/>
+                <state_interface name="velocity"/>
             </joint>
             <joint name="joint_5">
                 <command_interface name="position"/>
-                <command_interface name="effort"/>
                 <state_interface name="position">
+                  <param name="initial_value">${initial_positions['joint_5']}</param>
                 </state_interface>
-                <state_interface name="effort"/>
+                <state_interface name="velocity"/>
+            </joint>
+            <joint name="joint_6">
+                <command_interface name="position"/>
+                <state_interface name="position">
+                  <param name="initial_value">${initial_positions['joint_6']}</param>
+                </state_interface>
+                <state_interface name="velocity"/>
             </joint>
         </ros2_control>

File: src/arm_moveit_config/config/ar3.urdf.xacro (robot description, xacro)
@@ -1,8 +1,9 @@
 <?xml version="1.0"?>
 <robot xmlns:xacro="http://www.ros.org/wiki/xacro" name="ar3">
+    <xacro:arg name="initial_positions_file" default="initial_positions.yaml" />
     <!-- Import ar3 urdf file -->
     <xacro:include filename="$(find arm_description)/urdf/ar3_moveit.urdf" />
     <!-- Import control_xacro -->
     <xacro:include filename="ar3.ros2_control.xacro" />
-    <xacro:ar3_ros2_control name="ArmGazeboSystem"/>
+    <xacro:ar3_ros2_control name="FakeSystem" initial_positions_file="$(arg initial_positions_file)"/>
 </robot>
