Commit message: 现在可以通过rviz2界面控制gazebo里的机械臂。修改了之前README里的错误

File: src/arm_description/urdf/ar3_moveit.urdf (robot description, URDF)
Before this commit: robot ar3, 9 links, 8 joints
Links:
- link base_link: geometry collision mesh filename=file://$(find arm_description)/meshes/base_link.STL; visual mesh filename=file://$(find arm_description)/meshes/base_link.STL
- link link_1: geometry collision mesh filename=file://$(find arm_description)/meshes/link_1.STL; visual mesh filename=file://$(find arm_description)/meshes/link_1.STL
- link link_2: geometry collision mesh filename=file://$(find arm_description)/meshes/link_2.STL; visual mesh filename=file://$(find arm_description)/meshes/link_2.STL
- link link_3: geometry collision mesh filename=file://$(find arm_description)/meshes/link_3.STL; visual mesh filename=file://$(find arm_description)/meshes/link_3.STL
- link link_4: geometry collision mesh filename=file://$(find arm_description)/meshes/link_4.STL; visual mesh filename=file://$(find arm_description)/meshes/link_4.STL
- link link_5: geometry collision mesh filename=file://$(find arm_description)/meshes/link_5.STL; visual mesh filename=file://$(find arm_description)/meshes/link_5.STL
- link link_6: geometry collision mesh filename=file://$(find arm_description)/meshes/link_6.STL; visual mesh filename=file://$(find arm_description)/meshes/link_6.STL

Commit message: 末端换成连接球释放自由度尝试

File: src/arm_description/urdf/ar3_moveit.urdf (robot description, URDF)
Before this commit: robot ar3, 9 links, 8 joints
Links:
- added link ball_link_x, mass 0.001; collision sphere radius=0.01; visual sphere radius=0.01
- added link ball_link_y, mass 0.001; collision sphere radius=0.01; visual sphere radius=0.01
- added link ball_link_z, mass 0.001; collision sphere radius=0.01; visual sphere radius=0.01
Joints:
- added joint ball_joint_x: type continuous, parent link_6, child ball_link_x, origin xyz=0 0 0 rpy=0 0 0, axis 1 0 0
- added joint ball_joint_y: type continuous, parent ball_link_x, child ball_link_y, origin xyz=0 0 0 rpy=0 0 0, axis 0 1 0
- added joint ball_joint_z: type continuous, parent ball_link_y, child ball_link_z, origin xyz=0 0 0 rpy=0 0 0, axis 0 0 1
- joint camera_joint: parent link_6 -> ball_link_z

File: src/arm_moveit_config/config/ar3.ros2_control.xacro (robot description, xacro)
@@ -51,4 +51,22 @@
                 <state_interface name="velocity"/>
             </joint>
+            <joint name="ball_joint_x">
+                <state_interface name="position">
+                  <param name="initial_value">${initial_positions['ball_joint_x']}</param>
+                </state_interface>
+                <state_interface name="velocity"/>
+            </joint>
+            <joint name="ball_joint_y">
+                <state_interface name="position">
+                  <param name="initial_value">${initial_positions['ball_joint_y']}</param>
+                </state_interface>
+                <state_interface name="velocity"/>
+            </joint>
+            <joint name="ball_joint_z">
+                <state_interface name="position">
+                  <param name="initial_value">${initial_positions['ball_joint_z']}</param>
+                </state_interface>
+                <state_interface name="velocity"/>
+            </joint>
         </ros2_control>
     </xacro:macro>
